Commit message: basic sitting pose for human

File: assistive_gym/envs/assets/primitives/plane_chair.urdf (robot description, URDF)
Before this commit: robot plane_chair, 1 links, 0 joints
Links:
- link planeChairLink: geometry collision box size=30 30 10; collision mesh filename=plane.obj scale=0.075 0.25 1
